Commit message: feat: Improve vis demos

File: resources/test_robot.urdf (robot description, URDF)
Before this commit: robot test_robot, 4 links, 3 joints
Links:
- removed link end_effector
- removed link link1
- removed link link2
- added link base, mass 0.0
- added link ee_link, mass 0.0; collision box size=0.01 0.01 0.01
- added link forearm_link, mass 3.87; collision mesh filename=ur10/collision/forearm.stl
- added link shoulder_link, mass 7.778; collision mesh filename=ur10/collision/shoulder.stl
- added link tool0, mass 0.0
- added link upper_arm_link, mass 12.93; collision mesh filename=ur10/collision/upperarm.stl
- added link world
- added link wrist_1_link, mass 1.96; collision mesh filename=ur10/collision/wrist1.stl
- added link wrist_2_link, mass 1.96; collision mesh filename=ur10/collision/wrist2.stl
- added link wrist_3_link, mass 0.202; collision mesh filename=ur10/collision/wrist3.stl
- link base_link: mass None -> 4.0; geometry collision mesh filename=ur10/collision/base.stl
Joints:
- removed joint base_to_link1
- removed joint link1_to_link2
- removed joint link2_to_end_effector
- added joint base_link-base_fixed_joint: type fixed, parent base_link, child base, origin xyz=0 0 0 rpy=0 0 -3.14159265359
- added joint ee_fixed_joint: type fixed, parent wrist_3_link, child ee_link, origin xyz=0.0 0.0922 0.0 rpy=0.0 0.0 1.57079632679
- added joint elbow_joint: type revolute, parent upper_arm_link, child forearm_link, origin xyz=0.0 -0.1719 0.612 rpy=0.0 0.0 0.0, axis 0 1 0, limit lower=-3.14159265359 upper=3.14159265359 effort=150.0 velocity=3.15
- added joint shoulder_lift_joint: type revolute, parent shoulder_link, child upper_arm_link, origin xyz=0.0 0.220941 0.0 rpy=0.0 1.57079632679 0.0, axis 0 1 0, limit lower=-6.28318530718 upper=6.28318530718 effort=330.0 velocity=2.16
- added joint shoulder_pan_joint: type revolute, parent base_link, child shoulder_link, origin xyz=0.0 0.0 0.1273 rpy=0.0 0.0 0.0, axis 0 0 1, limit lower=-6.28318530718 upper=6.28318530718 effort=330.0 velocity=2.16
- added joint world_joint: type fixed, parent world, child base_link, origin xyz=0.0 0.0 0.0 rpy=0.0 0.0 0.0
- added joint wrist_1_joint: type revolute, parent forearm_link, child wrist_1_link, origin xyz=0.0 0.0 0.5723 rpy=0.0 1.57079632679 0.0, axis 0 1 0, limit lower=-6.28318530718 upper=6.28318530718 effort=54.0 velocity=3.2
- added joint wrist_2_joint: type revolute, parent wrist_1_link, child wrist_2_link, origin xyz=0.0 0.1149 0.0 rpy=0.0 0.0 0.0, axis 0 0 1, limit lower=-6.28318530718 upper=6.28318530718 effort=54.0 velocity=3.2
- added joint wrist_3_joint: type revolute, parent wrist_2_link, child wrist_3_link, origin xyz=0.0 0.0 0.1157 rpy=0.0 0.0 0.0, axis 0 1 0, limit lower=-6.28318530718 upper=6.28318530718 effort=54.0 velocity=3.2
- added joint wrist_3_link-tool0_fixed_joint: type fixed, parent wrist_3_link, child tool0, origin xyz=0 0.0922 0 rpy=-1.57079632679 0 0
